File: hw/wulpus_pro_acq_pcb/hv_mux_tr_sw.kicad_sch (KiCad schematic)
At the start: 40 parts, among them J1 DF40C-40DS-0.4V(51), J2 DF40C-40DS-0.4V(51), J3 91931-31169LF, J4 DF52-16S-0.8H(21), J5 91931-31169LF, J6 DF52-16S-0.8H(21), J7 Solder Jumper, J8 Solder Jumper, J9 Solder Jumper, U11 HV2707T-C/R8X, U12 TPS22916CYFPR, U13 MD0100N8-G

Commit message: Cleaned teh project, removen eval board components
Parts:
- removed C34, C35, C36, C37: 2.2 uF 50V, FP-GRM188-0_2-IPC_B, symbol Altium Content Vault:U_hv_mux_tr_sw_0_11868f565c42a9108669ba33697ecf6_Altium Co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
- removed J3, J5: 91931-31169LF, cmut_conn.PcbLib:FRAMETOME_91931-31169LF, symbol cmut_conn:U_hv_mux_tr_sw_0_91931-31169LF_cmut_conn.SCHLIB
- removed J4, J6: DF52-16S-0.8H(21), CONN_DF52-16S-0.8H(21)_HIR, symbol wulpus_hv:U_hv_mux_tr_sw_0_mirrored_DF52-16S-0.8H(21)_wulpus_hv.SCHLIB
- removed TP14, TP15: TP-SM-C-100, TP-SM-C-100, symbol wulpus:U_hv_mux_tr_sw_1_CMP-0484-00002-1_wulpus.SCHLIB
- removed TP16, TP17: TP-SM-C-100, TP-SM-C-100, symbol wulpus:U_hv_mux_tr_sw_2_CMP-0484-00002-1_wulpus.SCHLIB
Connections:
- no-connect marks 137 -> 15
Other:
- note removed: "Off-board Connectors"
