File: hw/wulpus_pro_acq_pcb/msp430.kicad_sch (KiCad schematic)
At the start: 36 parts, among them J10 U.FL-R-SMT-1(10), J11 U.FL-R-SMT-1(10), U14 MSP430FR5043IRGCT, X2 FY0800018, Y1 AWSCR-8.00CV-T, Y2 ABS05-32.768KHZ-9-T

Commit message: Cleaned teh project, removen eval board components
Parts:
- removed PJ1: 5051100892, MOLEX_5051100892, symbol wulpus:U_msp430_0_mirrored_MOLEX_5051100892_wulpus.SCHLIB
Connections:
- net BSL_UART_RX: no longer names the net of U14.22 (P2.1_UCA1STE_UCA3SOMI_UCA3RXD)
- net BSL_UART_TX: no longer names the net of U14.21 (P2.0_UCA1CLK_UCA3SIMO_UCA3TXD)
- no-connect marks 4 -> 6
Other:
- note removed: "BSL Signals"
