File: hw/wulpus_pro_acq_pcb/wulpus_pro_acq_pcb.kicad_sch (KiCad schematic)
At the start: 7 parts, among them M1 Mounting Hole, M2 Mounting Hole, M3 Mounting Hole, M4 Mounting Hole

Commit message: Cleaned teh project, removen eval board components
Parts:
- removed A1: Logo ETH Zurich, eth-zurich_3mm, symbol ETHZ Vault:root_0_Logo ETH Zurich_ETHZ Vault
- removed M1, M2, M3, M4: Mounting Hole, Mounting Hole, symbol ETHZ Vault:root_3_Hole_ETHZ Vault
Connections:
- no-connect marks 4 -> 0
Other:
- sheet U_host_connector ports: added none; removed MSP430_BSL{BSL_UART}
- sheet U_msp430 ports: added none; removed MSP430_BSL{BSL_UART}
