File: hw/wulpus_wifi_host_pcb/wulpus_pro_conn.kicad_sch (KiCad schematic)
At the start: 1 part, among them J2 DF40C-50DP-0.4V_51_

Commit message: Updated footprints, mapped 3D models, added layerstack, partial placement and layout
Parts:
- added C7, C8: 10 uF, Capacitor_SMD:C_0402_1005Metric, symbol Device:C
- added TP4: TestPoint, TestPoint:TestPoint_Pad_1.0x1.0mm, symbol Connector:TestPoint
Connections:
- net SPI.MOSI: now reaches J2.1
- net GND: now reaches J2.15
- net GND: now also J2.16, J2.36, C7.2, C8.2
- net SPI.MISO: now reaches J2.2
- net MSP_JTAG.TEST: now reaches J2.22
- net at J2.24: now also TP4.1
- net data_rdy: now reaches J2.25
- net MSP_JTAG.TDO: now reaches J2.26
- net MSP_JTAG.TDI: now reaches J2.28
- net +3V3: now reaches J2.29
- net +3V3: now also J2.31, C8.1
- net SPI.SS: now reaches J2.3
- net MSP_JTAG.TMS: now reaches J2.30
- net +5V: now reaches J2.33
- net +3V3 ESP: now reaches J2.37
- net +3V3 ESP: now also J2.39
- net SPI.CLK: now reaches J2.4
- net +V_board: now reaches J2.47
- net +V_board: now also J2.49, C7.1
- net MSP_JTAG.TCK: now reaches J2.48
- net MSP_JTAG.RST_n: now reaches J2.50
- no-connect marks 0 -> 28
Other:
- note added: "Board 2 Board Connector"
- note added: "JTAG and SPI buses"
- moved on the sheet: J2

Commit message: Finished layout, fixed DRCs
Parts:
- added TP6, TP7: TestPoint, TestPoint:TestPoint_Pad_1.0x1.0mm, symbol Connector:TestPoint
Connections:
- net GND: now also TP6.1, TP7.1
Other:
- note added: "GND Test Points"

Commit message: Changed cap footprints to 0603
Parts:
- C7, C8: footprint Capacitor_SMD:C_0402_1005Metric -> Capacitor_SMD:C_0603_1608Metric
- TP4, TP6, TP7: now left out of the parts list
Changed lines of the file:
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@@
 			)
 		)
-		(property "Footprint" "Capacitor_SMD:C_0402_1005Metric"
+		(property "Footprint" "Capacitor_SMD:C_0603_1608Metric"
 			(at 138.1252 119.38 0)
 			(hide yes)
@@
 			)
 		)
-		(property "Footprint" "Capacitor_SMD:C_0402_1005Metric"
+		(property "Footprint" "Capacitor_SMD:C_0603_1608Metric"
 			(at 157.1752 119.38 0)
 			(hide yes)
@@
 		(body_style 1)
 		(exclude_from_sim no)
-		(in_bom yes)
+		(in_bom no)
 		(on_board yes)
 		(in_pos_files yes)
@@
 		(body_style 1)
 		(exclude_from_sim no)
-		(in_bom yes)
+		(in_bom no)
 		(on_board yes)
 		(in_pos_files yes)
@@
 		(body_style 1)
 		(exclude_from_sim no)
-		(in_bom yes)
-		(on_board yes)
-		(in_pos_files yes)
+		(in_bom no)
+		(on_board yes)
+		(in_pos_files yes)

Commit message: Fixed BOM, added jobset file, regenerated fabrication outputs
Parts:
- C7, C8: MANUFACTURER (none) -> Murata Electronics; MP (none) -> GRM188R61A106ME69
Changed lines of the file:
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@@
+			)
+		)
+		(property "MANUFACTURER" "Murata Electronics"
+			(at 137.16 115.57 0)
+			(hide yes)
+			(show_name no)
+			(do_not_autoplace no)
+			(effects
+				(font
+					(size 1.27 1.27)
+				)
+			)
+		)
+		(property "MP" "GRM188R61A106ME69"
+			(at 137.16 115.57 0)
+			(hide yes)
+			(show_name no)
+			(do_not_autoplace no)
+			(effects
+				(font
+					(size 1.27 1.27)
+				)
 			)
 		)
@@
 			(at 156.21 115.57 0)
 			(hide yes)
+			(show_name no)
+			(do_not_autoplace no)
+			(effects
+				(font
+					(size 1.27 1.27)
+				)
+			)
+		)
+		(property "MANUFACTURER" "Murata Electronics"
+			(at 156.21 115.57 0)
+			(hide yes)
+			(show_name no)
+			(do_not_autoplace no)
+			(effects
+				(font
+					(size 1.27 1.27)
+				)
+			)
+		)
+		(property "MP" "GRM188R61A106ME69"
+			(at 156.21 115.57 0)
+			(hide yes)

Commit message: Added out capacitors for DC-DCs, regenerated fabrication files
Parts:
- renumbered C8 to C10, C7 to C9, TP6 to TP5, TP7 to TP6, TP4 to TP7
Changed lines of the file:
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@@
 		(dnp no)
 		(fields_autoplaced yes)
-		(property "Reference" "#PWR031"
+		(property "Reference" "#PWR037"
 			(at 156.21 125.73 0)
 			(hide yes)
@@
 			(project "wulpus_pro_wifi_host"
 				(path "/939c1465-135d-46db-aee7-7d874dab9895/b091b669-3a93-4e17-8613-2d1df892afc8"
-					(reference "#PWR031")
+					(reference "#PWR037")
 					(unit 1)
 				)
@@
 		(dnp no)
 		(fields_autoplaced yes)
-		(property "Reference" "#PWR033"
+		(property "Reference" "#PWR039"
 			(at 187.96 78.74 0)
 			(hide yes)
@@
 			(project "wulpus_pro_wifi_host"
 				(path "/939c1465-135d-46db-aee7-7d874dab9895/b091b669-3a93-4e17-8613-2d1df892afc8"
-					(reference "#PWR033")
+					(reference "#PWR039")
 					(unit 1)
 				)
@@
 		(dnp no)
 		(fields_autoplaced yes)
-		(property "Reference" "#PWR040"
+		(property "Reference" "#PWR033"
 			(at 82.55 181.61 0)
 			(hide yes)
@@
 			(project "wulpus_pro_wifi_host"
 				(path "/939c1465-135d-46db-aee7-7d874dab9895/b091b669-3a93-4e17-8613-2d1df892afc8"
-					(reference "#PWR040")
+					(reference "#PWR033")
 					(unit 1)
 				)
@@
 		(dnp no)
 		(fields_autoplaced yes)
-		(property "Reference" "#PWR039"
+		(property "Reference" "#PWR032"
 			(at 66.04 181.61 0)
 			(hide yes)
@@
 			(project "wulpus_pro_wifi_host"
 				(path "/939c1465-135d-46db-aee7-7d874dab9895/b091b669-3a93-4e17-8613-2d1df892afc8"
-					(reference "#PWR039")
+					(reference "#PWR032")
 					(unit 1)
 				)
@@
 		(dnp no)
 		(fields_autoplaced yes)
-		(property "Reference" "#PWR037"
+		(property "Reference" "#PWR043"
 			(at 236.22 83.82 0)
 			(hide yes)
@@
 			(project "wulpus_pro_wifi_host"
 				(path "/939c1465-135d-46db-aee7-7d874dab9895/b091b669-3a93-4e17-8613-2d1df892afc8"
-					(reference "#PWR037")
+					(reference "#PWR043")
 					(unit 1)
 				)
@@
 		(in_pos_files yes)
 		(dnp no)
-		(property "Reference" "#PWR028"
+		(property "Reference" "#PWR034"
 			(at 137.16 115.57 0)
 			(hide yes)
@@
 			(project "wulpus_pro_wifi_host"
 				(path "/939c1465-135d-46db-aee7-7d874dab9895/b091b669-3a93-4e17-8613-2d1df892afc8"
-					(reference "#PWR028")
+					(reference "#PWR034")
 					(unit 1)
 				)
@@
 		(dnp no)
 		(fields_autoplaced yes)
-		(property "Reference" "C7"
+		(property "Reference" "C9"
 			(at 140.97 114.2999 0)
 			(show_name no)
@@
 			(project "wulpus_pro_wifi_host"
 				(path "/939c1465-135d-46db-aee7-7d874dab9895/b091b669-3a93-4e17-8613-2d1df892afc8"
-					(reference "C7")
+					(reference "C9")
 					(unit 1)
 				)
@@
 		(in_pos_files yes)
 		(dnp no)
-		(property "Reference" "#PWR030"
+		(property "Reference" "#PWR036"
 			(at 156.21 115.57 0)
 			(hide yes)
@@
 			(project "wulpus_pro_wifi_host"
 				(path "/939c1465-135d-46db-aee7-7d874dab9895/b091b669-3a93-4e17-8613-2d1df892afc8"
-					(reference "#PWR030")
+					(reference "#PWR036")
 					(unit 1)
 				)
@@
 		(dnp no)
 		(fields_autoplaced yes)
-		(property "Reference" "#PWR036"
+		(property "Reference" "#PWR042"
 			(at 180.34 109.22 0)
 			(hide yes)
@@
 			(project "wulpus_pro_wifi_host"
 				(path "/939c1465-135d-46db-aee7-7d874dab9895/b091b669-3a93-4e17-8613-2d1df892afc8"
-					(reference "#PWR036")
+					(reference "#PWR042")
 					(unit 1)
 				)
@@
 		(dnp no)
 		(fields_autoplaced yes)
-		(property "Reference" "#PWR038"
+		(property "Reference" "#PWR044"
 			(at 236.22 109.22 0)
 			(hide yes)
@@
 			(project "wulpus_pro_wifi_host"
 				(path "/939c1465-135d-46db-aee7-7d874dab9895/b091b669-3a93-4e17-8613-2d1df892afc8"
-					(reference "#PWR038")
+					(reference "#PWR044")
 					(unit 1)
 				)
@@
 		(dnp no)
 		(fields_autoplaced yes)
-		(property "Reference" "C8"
+		(property "Reference" "C10"
 			(at 160.02 114.2999 0)
 			(show_name no)
@@
 			(project "wulpus_pro_wifi_host"
 				(path "/939c1465-135d-46db-aee7-7d874dab9895/b091b669-3a93-4e17-8613-2d1df892afc8"
-					(reference "C8")
+					(reference "C10")
 					(unit 1)
 				)
@@
 		(in_pos_files yes)
 		(dnp no)
-		(property "Reference" "TP6"
+		(property "Reference" "TP5"
 			(at 66.294 168.656 90)
 			(show_name no)
@@
 			(project "wulpus_pro_wifi_host"
 				(path "/939c1465-135d-46db-aee7-7d874dab9895/b091b669-3a93-4e17-8613-2d1df892afc8"
-					(reference "TP6")
+					(reference "TP5")
 					(unit 1)
 				)
@@
 		(in_pos_files yes)
 		(dnp no)
-		(property "Reference" "TP4"
+		(property "Reference" "TP7"
 			(at 249.174 99.314 90)
 			(show_name no)
@@
 			(project "wulpus_pro_wifi_host"
 				(path "/939c1465-135d-46db-aee7-7d874dab9895/b091b669-3a93-4e17-8613-2d1df892afc8"
-					(reference "TP4")
+					(reference "TP7")
 					(unit 1)
 				)
@@
 		(in_pos_files yes)
 		(dnp no)
-		(property "Reference" "#PWR032"
+		(property "Reference" "#PWR038"
 			(at 181.61 68.58 0)
 			(hide yes)
@@
 			(project "wulpus_pro_wifi_host"
 				(path "/939c1465-135d-46db-aee7-7d874dab9895/b091b669-3a93-4e17-8613-2d1df892afc8"
-					(reference "#PWR032")
+					(reference "#PWR038")
 					(unit 1)
 				)
@@
 		(dnp no)
 		(fields_autoplaced yes)
-		(property "Reference" "#PWR035"
+		(property "Reference" "#PWR041"
 			(at 187.96 91.44 0)
 			(hide yes)
@@
 			(project "wulpus_pro_wifi_host"
 				(path "/939c1465-135d-46db-aee7-7d874dab9895/b091b669-3a93-4e17-8613-2d1df892afc8"
-					(reference "#PWR035")
+					(reference "#PWR041")
 					(unit 1)
 				)
@@
 		(dnp no)
 		(fields_autoplaced yes)
-		(property "Reference" "#PWR029"
+		(property "Reference" "#PWR035"
 			(at 137.16 125.73 0)
 			(hide yes)
@@
 			(project "wulpus_pro_wifi_host"
 				(path "/939c1465-135d-46db-aee7-7d874dab9895/b091b669-3a93-4e17-8613-2d1df892afc8"
-					(reference "#PWR029")
+					(reference "#PWR035")
 					(unit 1)
 				)
@@
 		(dnp no)
 		(fields_autoplaced yes)
-		(property "Reference" "#PWR034"
+		(property "Reference" "#PWR040"
 			(at 187.96 86.36 0)
 			(hide yes)
@@
 			(project "wulpus_pro_wifi_host"
 				(path "/939c1465-135d-46db-aee7-7d874dab9895/b091b669-3a93-4e17-8613-2d1df892afc8"
-					(reference "#PWR034")
+					(reference "#PWR040")
 					(unit 1)
 				)
@@
 		(in_pos_files yes)
 		(dnp no)
-		(property "Reference" "TP7"
+		(property "Reference" "TP6"
 			(at 82.804 168.656 90)
 			(show_name no)
@@
 			(project "wulpus_pro_wifi_host"
 				(path "/939c1465-135d-46db-aee7-7d874dab9895/b091b669-3a93-4e17-8613-2d1df892afc8"
-					(reference "TP7")
-					(unit 1)
-				)
+					(reference "TP6")
+					(unit 1)
+				)

Commit message: Rename project to WULPUS Pro Max
- update user-facing branding across documentation, firmware, and software
- update repository URLs while preserving compatibility identifiers
- release WiFi host PCB v1.0.1 with revised metadata and silkscreen
- regenerate hardware design and fabrication outputs
Other:
- title: (none) -> WULPUS Pro Max WiFi host
Changed lines of the file:
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@@
 	(generator_version "10.0")
 	(paper "A4")
+	(title_block
+		(title "WULPUS Pro Max WiFi host")
+		(rev "v1.0.1")
+		(comment 1 "Reviewer: Cedric Hirschi")
+		(comment 2 "Author: Sergei Vostrikov")
+	)
 	(rectangle
 		(start 125.73 39.37)
