File: hw/wulpus_wifi_host_pcb/wulpus_pro_wifi_host.kicad_pcb (KiCad board)
At the start: 4 copper layers, 39 x 21 mm, 52 parts, among them J1 S2B-PH-SM4-TB_LF__SN_, J2 DF40C-50DP-0.4V_51_, Q1 FS8205A, Q2 LP0404N3T5G, U1 XIAO-ESP32-C6-SMD, U2 TPS63900DSKR, U3 BQ29700DSER, U4 TPS63900DSKR

Commit message: Rename project to WULPUS Pro Max
- update user-facing branding across documentation, firmware, and software
- update repository URLs while preserving compatibility identifiers
- release WiFi host PCB v1.0.1 with revised metadata and silkscreen
- regenerate hardware design and fabrication outputs
Other:
- board text added: "WiFi Host Board v1.0.1 Sergei Vostrikov 21.09.26"
- board text removed: "WiFi Host Board v1.0 Sergei Vostrikov 30.07.26"
Changed lines of the file:
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@@
 	(paper "A4")
 	(title_block
-		(title "WULPUS PRO WiFi host ")
-		(date "2026-08-22")
-		(rev "v1.0.0")
-		(comment 1 "Reviewer: Cedric Hirshi")
+		(title "WULPUS Pro Max WiFi host ")
+		(date "2026-09-21")
+		(rev "v1.0.1")
+		(comment 1 "Reviewer: Cedric Hirschi")
 		(comment 2 "Author: Sergei Vostrikov")
 	)
@@
 		(layer "Edge.Cuts")
 	)
-	(gr_text "WiFi Host Board v1.0\nSergei Vostrikov\n30.07.26"
-		(at 102.23 99.95 0)
+	(gr_text "WiFi Host Board v1.0.1\nSergei Vostrikov\n21.09.26"
+		(at 102.825 100.15 0)
 		(layer "B.SilkS")
 		(effects
